File: src/PCI_COMPLETA_1.0/PCI_COMPLETA_1.0.kicad_pcb (KiCad board)
At the start: 4 copper layers, 54.6 x 42.5 mm, 46 parts, among them J1 USB_B_Micro, J2 Conn_01x06_Socket, J3 USB_B_Micro, J4 Screw_Terminal_01x02, J5 Screw terminal for switch, Q1 FS8205, SW1 RESET1, SW2 BOOT1, U1 ESP32-S3-MINI-1, U2 MPU-9250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

Commit message: fix: corrige envio de valores de angulo
Parts:
- removed C10, C11: 0,1uF, Capacitor_SMD:C_0603_1608Metric
- removed C12: 10nF, Capacitor_SMD:C_0603_1608Metric
- removed U3: D3V3XA4B10LP, Package_DFN_QFN:Diodes_UDFN-10_1.0x2.5mm_P0.5mm
- added C13: 2.2nF 50V, Capacitor_SMD:C_0603_1608Metric, F.Cu at (85.1, 125.2)
- added C14: 0.1µF 2V, Capacitor_SMD:C_0603_1608Metric, F.Cu at (84.3, 132.8)
- added C15: 10nF 4V, Capacitor_SMD:C_0603_1608Metric, F.Cu at (87.4, 132.1)
- added C16: 0.1µF 4V, Capacitor_SMD:C_0603_1608Metric, F.Cu at (89.4, 132.1)
- added R15: 22, Resistor_SMD:R_0402_1005Metric, F.Cu at (67.0, 126.1)
- added R16: 22, Resistor_SMD:R_0402_1005Metric, F.Cu at (68.1, 126.1)
- added R17: 10K, Resistor_SMD:R_0603_1608Metric, F.Cu at (70.3, 133.2)
- added U8: MPU-6050, Sensor_Motion:InvenSense_QFN-24_4x4mm_P0.5mm, F.Cu at (83.2, 129.2)
- U2: value MPU-9250 -> ESD7104MUTAG; footprint Sensor_Motion:InvenSense_QFN-24_3x3mm_P0.4mm -> footprints:UDFN10_ONS
- moved U2 21.2 mm to (68.3, 145.4), turned to 90 degrees
Connections:
- J1 pad 2: /USB_N -> /IN_N
- J1 pad 3: /USB_P -> /IN_P
- U2 pad 1: /3V3 -> /IN_N
- U2 pad 10: Net-(U2-REGOUT) -> /IN_N
- U2 pad 2: (no net) -> /IN_P
- U2 pad 3: (no net) -> OUT-
- U2 pad 4: (no net) -> VIN
- U2 pad 5: (no net) -> unconnected-(U2-I/O-Pad5)
- U2 pad 6: (no net) -> unconnected-(U2-NC-Pad6)
- U2 pad 7: unconnected-(U2-AUX_CL-Pad7) -> VIN
- U2 pad 8: /3V3 -> OUT-
- U2 pad 9: unconnected-(U2-AD0/MISO-Pad9) -> /IN_P
Routing:
- net /USB_P: track 23.8 -> 1.56 mm
- net /USB_N: track 23.7 -> 1.53 mm
- net /IN_N: track 0.00 -> 21.5 mm
- net /IN_P: track 0.00 -> 21.5 mm
- net /3V3: track 152.6 -> 145.9 mm
- net Net-(U2-REGOUT): track 4.20 -> 0.00 mm
- net /GPIO_0: track 44.7 -> 47.2 mm, vias 2 -> 3
- net Net-(U8-CPOUT): track 0.00 -> 2.24 mm
- net /SDA: track 60.2 -> 58.0 mm
- net Net-(U8-REGOUT): track 0.00 -> 1.69 mm
- net /SCL: track 46.3 -> 44.6 mm
- net OUT-: track 13.8 -> 12.6 mm, vias 115 -> 113
- net VIN: track 94.2 -> 93.5 mm
Other:
- board size 54.6 x 42.5 mm -> 56.7 x 42.5 mm
